File: hw_platform/ADS1292EMG2x/analog_frontend.kicad_sch (KiCad schematic)
At the start: 17 parts

Commit message: working on schematic
Other:
- company: (none) -> Developed by Rf-lab.org
- title: (none) -> EMG-2x: Two channel EMG board
Changed lines of the file:
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@@
 (kicad_sch (version 20211123) (generator eeschema)
   (paper "A4")
+  (title_block
+    (title "EMG-2x: Two channel EMG board")
+    (date "2022-02-11")
+    (rev "1")
+    (company "Developed by Rf-lab.org")
+  )
   (junction (at 71.12 29.21) (diameter 0) (color 0 0 0 0)
   )

Commit message: schematic verification
Parts:
- added R5: 1M, Resistor_SMD:R_0805_2012Metric_Pad1.20x1.40mm_HandSolder, symbol Device:R
Connections:
- net INA_Vref: now also R5.1
- net at R?.2, U?.5 (Ref): now also R5.2
