File: hw_platform/ADS1292EMG2x/power_supply.kicad_sch (KiCad schematic)
At the start: 10 parts

Commit message: working on schematic
Parts:
- added R? (x2): 10k, symbol Device:R_US
Connections:
- net GND: now also R?.1
- net at C?.1, J?.1 (Pin_1), Q?.2 (S)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: now also R?.2
- new net BAT_MON: R?.1, R?.2
Other:
- company: (none) -> Developed by Rf-lab.org
- title: (none) -> EMG-2x: Two channel EMG board
Changed lines of the file:
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@@
 (kicad_sch (version 20211123) (generator eeschema)
   (paper "A4")
+  (title_block
+    (title "EMG-2x: Two channel EMG board")
+    (date "2022-02-11")
+    (rev "1")
+    (company "Developed by Rf-lab.org")
+  )
   (junction (at 111.76 72.39) (diameter 0) (color 0 0 0 0)
   )
@@
   (junction (at 186.69 72.39) (diameter 0) (color 0 0 0 0)
   )
+  (junction (at 170.18 100.33) (diameter 0) (color 0 0 0 0)
+  )
   (junction (at 165.1 72.39) (diameter 0) (color 0 0 0 0)
   )
@@
     (stroke (width 0) (type default) (color 0 0 0 0))
   )
+  (wire (pts (xy 170.18 100.33) (xy 170.18 101.6))
+    (stroke (width 0) (type default) (color 0 0 0 0))
+  )
   (wire (pts (xy 140.97 92.71) (xy 140.97 95.25))
     (stroke (width 0) (type default) (color 0 0 0 0))
@@
     (stroke (width 0) (type default) (color 0 0 0 0))
   )
+  (wire (pts (xy 170.18 110.49) (xy 170.18 109.22))
+    (stroke (width 0) (type default) (color 0 0 0 0))
+  )
   (wire (pts (xy 165.1 72.39) (xy 176.53 72.39))
     (stroke (width 0) (type default) (color 0 0 0 0))
@@
     (stroke (width 0) (type default) (color 0 0 0 0))
   )
+  (wire (pts (xy 170.18 91.44) (xy 170.18 87.63))
+    (stroke (width 0) (type default) (color 0 0 0 0))
+  )
   (wire (pts (xy 165.1 73.66) (xy 165.1 72.39))
     (stroke (width 0) (type default) (color 0 0 0 0))
@@
     (stroke (width 0) (type default) (color 0 0 0 0))
   )
+  (wire (pts (xy 170.18 99.06) (xy 170.18 100.33))
+    (stroke (width 0) (type default) (color 0 0 0 0))
+  )
   (wire (pts (xy 128.27 97.79) (xy 128.27 101.6))
     (stroke (width 0) (type default) (color 0 0 0 0))
@@
   (wire (pts (xy 138.43 87.63) (xy 148.59 87.63))
     (stroke (width 0) (type default) (color 0 0 0 0))
+  )
+  (wire (pts (xy 191.77 100.33) (xy 170.18 100.33))
+    (stroke (width 0) (type default) (color 0 0 0 0))
+  )
+  (hierarchical_label "BAT_MON" (shape output) (at 191.77 100.33 0)
+    (effects (font (size 1.27 1.27)) (justify left))
   )
   (hierarchical_label "VPWR" (shape output) (at 191.77 72.39 0)
@@
   (hierarchical_label "VUSB{slash}2.1A" (shape input) (at 106.68 72.39 180)
     (effects (font (size 1.27 1.27)) (justify right))
+  )
+  (symbol (lib_id "Device:R_US") (at 170.18 95.25 180) (unit 1)
+    (in_bom yes) (on_board yes)
+    (property "Reference" "R?" (id 0) (at 166.37 93.98 0)
+      (effects (font (size 1.27 1.27)) (justify right))
+    )
+    (property "Value" "10k" (id 1) (at 165.1 96.52 0)
+      (effects (font (size 1.27 1.27)) (justify right))
+    )
+    (property "Footprint" "" (id 2) (at 169.164 94.996 90)
+      (effects (font (size 1.27 1.27)) hide)
+    )
+    (property "Datasheet" "~" (id 3) (at 170.18 95.25 0)
+      (effects (font (size 1.27 1.27)) hide)
+    )
+    (pin "1")
+    (pin "2")
   )
   (symbol (lib_id "power:GND") (at 116.84 101.6 0) (unit 1)
@@
     )
     (property "Datasheet" "~" (id 3) (at 148.59 92.71 0)
+      (effects (font (size 1.27 1.27)) hide)
+    )
+    (pin "1")
+    (pin "2")
+  )
+  (symbol (lib_id "Device:R_US") (at 170.18 105.41 180) (unit 1)
+    (in_bom yes) (on_board yes)
+    (property "Reference" "R?" (id 0) (at 166.37 104.14 0)
+      (effects (font (size 1.27 1.27)) (justify right))
+    )
+    (property "Value" "10k" (id 1) (at 165.1 106.68 0)
+      (effects (font (size 1.27 1.27)) (justify right))
+    )
+    (property "Footprint" "" (id 2) (at 169.164 105.156 90)
+      (effects (font (size 1.27 1.27)) hide)
+    )
+    (property "Datasheet" "~" (id 3) (at 170.18 105.41 0)
       (effects (font (size 1.27 1.27)) hide)
     )
@@
       (effects (font (size 1.27 1.27)) hide)
     )
+    (pin "1")
+  )
+  (symbol (lib_id "power:GND") (at 170.18 110.49 0) (unit 1)
+    (in_bom yes) (on_board yes)
+    (property "Reference" "#PWR?" (id 0) (at 170.18 116.84 0)
+      (effects (font (size 1.27 1.27)) hide)
+    )
+    (property "Value" "GND" (id 1) (at 167.64 114.3 0)
+      (effects (font (size 1.27 1.27)) (justify left))
+    )
+    (property "Footprint" "" (id 2) (at 170.18 110.49 0)
+      (effects (font (size 1.27 1.27)) hide)
+    )
+    (property "Datasheet" "" (id 3) (at 170.18 110.49 0)
+      (effects (font (size 1.27 1.27)) hide)
+    )
