File: hw_platform/ADS1299EMG8xR2/ADS1299EMG8xR2.kicad_pcb (KiCad board)
At the start: 2 copper layers, 81 parts, among them U1 PJ-325-5P, U10 LM1117-5.0, U11 LM1117-3.3, U12 LM1117-5.0, U13 ESP32-DevKitC, U2 PJ-325-5P, U3 PJ-325-5P, U4 PJ-325-5P, U5 PJ-325-5P, U6 PJ-325-5P, U7 PJ-325-5P, U8 PJ-325-5P, U9 ADS1299

Commit message: partial routed
Parts:
- JP1, JP2, JP4, JP6: footprint Jumper:SolderJumper-3_P1.3mm_Bridged2Bar12_Pad1.0x1.5mm_NumberLabels -> Connector_PinHeader_2.54mm:PinHeader_1x03_P2.54mm_Vertical
- JP3, JP5: footprint Jumper:SolderJumper-2_P1.3mm_Bridged2Bar_Pad1.0x1.5mm -> Connector_PinHeader_2.54mm:PinHeader_1x02_P2.54mm_Vertical
- moved BT1 133.0 mm to (173.4, 70.9), turned to 270 degrees
- moved C30 89.8 mm to (160.2, 111.8), turned to 90 degrees
- moved C24 85.3 mm to (169.7, 111.9), turned to 270 degrees
- moved BT2 85.2 mm to (123.2, 70.3), turned to 90 degrees
- moved C18 83.4 mm to (182.4, 111.8), turned to 90 degrees
- moved C35 83.3 mm to (147.5, 111.9), turned to 270 degrees
- moved U12 79.9 mm to (153.8, 109.0), turned to 90 degrees
- moved U10 77.4 mm to (176.1, 109.0), turned to 90 degrees
- moved JP5 60.3 mm to (188.0, 99.7), turned to 180 degrees
- moved JP6 58.5 mm to (154.3, 95.2), turned to 270 degrees
- moved JP2 26.7 mm to (136.5, 26.7)
- moved R20 22.5 mm to (153.0, 83.0)
- moved JP1 17.5 mm to (141.6, 102.2), turned to 0 degrees
- moved R18 15.9 mm to (138.4, 33.3), turned to 90 degrees
- moved C26 13.2 mm to (156.7, 36.1)
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Routing:
- net Net-(C14-Pad2): track 0.00 -> 56.1 mm
- net Net-(C13-Pad2): track 0.00 -> 48.1 mm
- net Net-(C1-Pad1): track 0.00 -> 48.0 mm
- net Net-(C2-Pad2): track 0.00 -> 41.0 mm
- net Net-(C12-Pad1): track 0.00 -> 40.2 mm
- net +5VA: track 0.00 -> 39.0 mm
- net Net-(C3-Pad1): track 0.00 -> 37.7 mm
- net Net-(C14-Pad1): track 0.00 -> 36.2 mm
- net Net-(C11-Pad2): track 0.00 -> 34.9 mm
- net Net-(C11-Pad1): track 0.00 -> 33.9 mm
- net Net-(C4-Pad2): track 0.00 -> 30.4 mm
- net Net-(JP3-Pad2): track 0.00 -> 29.1 mm
- net Net-(C15-Pad2): track 0.00 -> 28.6 mm
- net +3V3: track 0.00 -> 27.7 mm
- net Net-(C5-Pad1): track 0.00 -> 26.5 mm
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Other:
- board outline added: 96 x 100 mm
- board text added: "BiasIn"
- board text added: "CRE"
- board text added: "EMG-8x Rev.2"
- board text added: "IN2"
- board text added: "IN3"
- board text added: "IN4"
- board text added: "IN5"
- board text added: "IN6"
- board text added: "IN7"
- board text added: "MGUPI/MIREA/KB3/KB2"
- board text added: "Rf-Lab.org"
- board text removed: "Common Reference electrode"

Commit message: REvision2_release
Parts:
- added R21: 10k, Resistor_SMD:R_0805_2012Metric_Pad1.20x1.40mm_HandSolder, F.Cu at (149.4, 69.1)
- added R22: 10k, Resistor_SMD:R_0805_2012Metric_Pad1.20x1.40mm_HandSolder, F.Cu at (149.3, 71.6)
- added REF**: OSHW-Logo2_14.6x12mm_SilkScreen, Symbol:OSHW-Logo2_14.6x12mm_SilkScreen, F.Cu at (131.1, 113.3)
- added REF**: KiCad-Logo2_5mm_SilkScreen, Symbol:KiCad-Logo2_5mm_SilkScreen, F.Cu at (174.0, 36.8)
- moved C42 5.87 mm to (151.4, 63.2), turned to 90 degrees
- moved JP1 5.28 mm to (136.4, 103.1), turned to 270 degrees
- moved R20 4.29 mm to (154.6, 87.0)
- moved R1 4.12 mm to (133.4, 97.5)
- moved C15 2.88 mm to (133.4, 93.7)
- moved C23 1.91 mm to (146.3, 78.7)
- moved C41 0.74 mm to (147.3, 65.8)
- moved C39 0.64 mm to (147.3, 62.9)
- moved C40 0.64 mm to (147.3, 60.3)
- moved C18 0.45 mm to (182.9, 111.9)
- moved C24 0.07 mm to (169.7, 111.9)
Connections:
- U13 pad 10: ADS_GPIO1 -> Net-(U13-Pad10)
- U13 pad 11: ADS_GPIO2 -> Net-(U13-Pad11)
- U9 pad 18: Net-(U9-Pad18) -> GNDA
- U9 pad 42: ADS_GPIO1 -> Net-(R22-Pad2)
- U9 pad 44: ADS_GPIO2 -> Net-(R21-Pad2)
- U9 pad 60: Net-(U9-Pad60) -> GNDA
Routing:
- net Net-(JP1-Pad3): track 0.00 -> 177.0 mm
- net +6V: track 0.00 -> 151.0 mm, vias 0 -> 1
- net +5VD: track 0.00 -> 134.2 mm
- net +5VA: track 39.0 -> 102.2 mm, vias 0 -> 1
- net Net-(JP1-Pad2): track 0.00 -> 52.8 mm
- net Net-(BT1-Pad2): track 0.00 -> 50.4 mm
- net ADS_~RESET: track 0.00 -> 47.7 mm
- net ADS_CLK: track 0.00 -> 46.9 mm
- net GNDD: track 0.00 -> 42.6 mm, vias 0 -> 6
- net +3V3: track 27.7 -> 65.9 mm
- net Net-(U13-Pad31): track 0.00 -> 34.1 mm
- net Net-(C24-Pad1): track 0.00 -> 34.0 mm
- net Net-(C35-Pad1): track 0.00 -> 31.0 mm
- net Net-(U13-Pad29): track 0.00 -> 29.6 mm
- net GNDA: track 0.00 -> 28.2 mm, vias 0 -> 8
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- added copper zone on B.Cu, net GNDA
- added copper zone on F.Cu, net GNDA
- added copper zone on B.Cu, net GNDD
- added copper zone on F.Cu, net GNDD
Other:
- net class Power_branch added: clearance 0.2, trace_width 1, via_dia 0.8, via_drill 0.4
- net class Power_bus added: clearance 0.2, trace_width 2, via_dia 0.8, via_drill 0.4
- board text added: "SRB1"
- board text removed: "CRE"

Commit message: revision 3
Parts:
- removed C1, C10, C11, C12, C15, C2, C6, C9: 4.7nF, Capacitor_SMD:C_0805_2012Metric_Pad1.18x1.45mm_HandSolder
- removed JP1, JP2: Jumper_3_Bridged12, Connector_PinHeader_2.54mm:PinHeader_1x03_P2.54mm_Vertical
- removed R10, R11, R13, R16, R17, R18, R9: 4.99k, Resistor_SMD:R_0805_2012Metric_Pad1.20x1.40mm_HandSolder
- removed U4, U5: PJ-325-5P, Connector_Audio:Jack_3.5mm_PJ-325-P5
- added C37: 470pF, Capacitor_SMD:C_0805_2012Metric_Pad1.18x1.45mm_HandSolder, F.Cu at (118.6, 56.9)
- added C38: 100nF, Capacitor_SMD:C_0805_2012Metric_Pad1.18x1.45mm_HandSolder, F.Cu at (117.8, 82.0)
- added C43: 100nF, Capacitor_SMD:C_0805_2012Metric_Pad1.18x1.45mm_HandSolder, F.Cu at (117.9, 71.6)
- added C46: 4.7nF, Capacitor_SMD:C_0805_2012Metric_Pad1.18x1.45mm_HandSolder, F.Cu at (121.7, 101.4)
- added C47: 4.7nF, Capacitor_SMD:C_0805_2012Metric_Pad1.18x1.45mm_HandSolder, F.Cu at (121.7, 95.8)
- added C48: 4.7nF, Capacitor_SMD:C_0805_2012Metric_Pad1.18x1.45mm_HandSolder, F.Cu at (118.4, 44.2)
- added C49: 4.7nF, Capacitor_SMD:C_0805_2012Metric_Pad1.18x1.45mm_HandSolder, F.Cu at (118.4, 39.6)
- added C50: 4.7nF, Capacitor_SMD:C_0805_2012Metric_Pad1.18x1.45mm_HandSolder, F.Cu at (121.7, 116.1)
- added C51: 4.7nF, Capacitor_SMD:C_0805_2012Metric_Pad1.18x1.45mm_HandSolder, F.Cu at (121.7, 111.0)
- added C52: 4.7nF, Capacitor_SMD:C_0805_2012Metric_Pad1.18x1.45mm_HandSolder, F.Cu at (118.4, 30.7)
- added C53: 4.7nF, Capacitor_SMD:C_0805_2012Metric_Pad1.18x1.45mm_HandSolder, F.Cu at (118.4, 26.1)
- added C54: 4.7nF, Capacitor_SMD:C_0805_2012Metric_Pad1.18x1.45mm_HandSolder, F.Cu at (115.1, 98.3)
- added C55: 4.7nF, Capacitor_SMD:C_0805_2012Metric_Pad1.18x1.45mm_HandSolder, F.Cu at (115.1, 41.9)
- added C56: 4.7nF, Capacitor_SMD:C_0805_2012Metric_Pad1.18x1.45mm_HandSolder, F.Cu at (115.3, 113.6)
- added C57: 4.7nF, Capacitor_SMD:C_0805_2012Metric_Pad1.18x1.45mm_HandSolder, F.Cu at (115.1, 28.7)
- added C58: 100nF, Capacitor_SMD:C_0805_2012Metric_Pad1.18x1.45mm_HandSolder, F.Cu at (132.6, 98.3)
- added C59: 100nF, Capacitor_SMD:C_0805_2012Metric_Pad1.18x1.45mm_HandSolder, F.Cu at (131.8, 41.9)
- added C60: 100nF, Capacitor_SMD:C_0805_2012Metric_Pad1.18x1.45mm_HandSolder, F.Cu at (132.1, 111.7)
- added C61: 100nF, Capacitor_SMD:C_0805_2012Metric_Pad1.18x1.45mm_HandSolder, F.Cu at (131.1, 32.0)
- added C62: 100nF, Capacitor_SMD:C_0805_2012Metric_Pad1.18x1.45mm_HandSolder, F.Cu at (134.6, 111.8)
- added C63: 100nF, Capacitor_SMD:C_0805_2012Metric_Pad1.18x1.45mm_HandSolder, F.Cu at (131.6, 28.7)
- added C64: 470pF, Capacitor_SMD:C_0805_2012Metric_Pad1.18x1.45mm_HandSolder, F.Cu at (122.2, 55.1)
- added R24: 220k, Resistor_SMD:R_0805_2012Metric_Pad1.20x1.40mm_HandSolder, F.Cu at (114.3, 54.1)
- added R25: 220k, Resistor_SMD:R_0805_2012Metric_Pad1.20x1.40mm_HandSolder, F.Cu at (114.3, 56.9)
- added R28: 220k, Resistor_SMD:R_0805_2012Metric_Pad1.20x1.40mm_HandSolder, F.Cu at (118.6, 51.3)
- added R29: 220k, Resistor_SMD:R_0805_2012Metric_Pad1.20x1.40mm_HandSolder, F.Cu at (118.6, 59.7)
- added R30: 220k, Resistor_SMD:R_0805_2012Metric_Pad1.20x1.40mm_HandSolder, F.Cu at (117.9, 78.5)
- added R31: 220k, Resistor_SMD:R_0805_2012Metric_Pad1.20x1.40mm_HandSolder, F.Cu at (117.9, 75.2)
- added R34: 4.99k, Resistor_SMD:R_0805_2012Metric_Pad1.20x1.40mm_HandSolder, F.Cu at (100.1, 92.5)
- added R35: 4.99k, Resistor_SMD:R_0805_2012Metric_Pad1.20x1.40mm_HandSolder, F.Cu at (99.1, 35.8)
- added R36: 4.99k, Resistor_SMD:R_0805_2012Metric_Pad1.20x1.40mm_HandSolder, F.Cu at (99.9, 106.9)
- added R37: 4.99k, Resistor_SMD:R_0805_2012Metric_Pad1.20x1.40mm_HandSolder, F.Cu at (100.1, 23.1)
- added R38: 4.99k, Resistor_SMD:R_0805_2012Metric_Pad1.20x1.40mm_HandSolder, F.Cu at (114.3, 102.1)
- added R39: 4.99k, Resistor_SMD:R_0805_2012Metric_Pad1.20x1.40mm_HandSolder, F.Cu at (114.3, 95.0)
- added R40: 4.99k, Resistor_SMD:R_0805_2012Metric_Pad1.20x1.40mm_HandSolder, F.Cu at (114.3, 45.2)
- added R41: 4.99k, Resistor_SMD:R_0805_2012Metric_Pad1.20x1.40mm_HandSolder, F.Cu at (114.3, 38.6)
- added R42: 1M, Resistor_SMD:R_0805_2012Metric_Pad1.20x1.40mm_HandSolder, F.Cu at (118.4, 116.1)
- added R43: 4.99k, Resistor_SMD:R_0805_2012Metric_Pad1.20x1.40mm_HandSolder, F.Cu at (114.3, 117.1)
- added R44: 4.99k, Resistor_SMD:R_0805_2012Metric_Pad1.20x1.40mm_HandSolder, F.Cu at (114.3, 110.0)
- added R45: 1M, Resistor_SMD:R_0805_2012Metric_Pad1.20x1.40mm_HandSolder, F.Cu at (121.2, 30.7)
- added R46: 4.99k, Resistor_SMD:R_0805_2012Metric_Pad1.20x1.40mm_HandSolder, F.Cu at (114.3, 32.0)
- added R47: 4.99k, Resistor_SMD:R_0805_2012Metric_Pad1.20x1.40mm_HandSolder, F.Cu at (114.3, 25.1)
- added R48: 1M, Resistor_SMD:R_0805_2012Metric_Pad1.20x1.40mm_HandSolder, F.Cu at (118.4, 101.3)
- added R49: 1M, Resistor_SMD:R_0805_2012Metric_Pad1.20x1.40mm_HandSolder, F.Cu at (121.2, 44.2)
- added R50: 1M, Resistor_SMD:R_0805_2012Metric_Pad1.20x1.40mm_HandSolder, F.Cu at (118.4, 95.8)
- added R51: 1M, Resistor_SMD:R_0805_2012Metric_Pad1.20x1.40mm_HandSolder, F.Cu at (121.2, 39.6)
- added R52: 1M, Resistor_SMD:R_0805_2012Metric_Pad1.20x1.40mm_HandSolder, F.Cu at (118.4, 111.0)
- added R53: 1M, Resistor_SMD:R_0805_2012Metric_Pad1.20x1.40mm_HandSolder, F.Cu at (121.2, 26.2)
- added R54: 100k, Resistor_SMD:R_0805_2012Metric_Pad1.20x1.40mm_HandSolder, F.Cu at (126.8, 102.9)
- added R55: 100k, Resistor_SMD:R_0805_2012Metric_Pad1.20x1.40mm_HandSolder, F.Cu at (125.7, 45.0)
- added R56: 100k, Resistor_SMD:R_0805_2012Metric_Pad1.20x1.40mm_HandSolder, F.Cu at (126.5, 117.3)
- added R57: 100k, Resistor_SMD:R_0805_2012Metric_Pad1.20x1.40mm_HandSolder, F.Cu at (125.5, 31.8)
- added R58: 100k, Resistor_SMD:R_0805_2012Metric_Pad1.20x1.40mm_HandSolder, F.Cu at (126.8, 95.2)
- added R59: 100k, Resistor_SMD:R_0805_2012Metric_Pad1.20x1.40mm_HandSolder, F.Cu at (125.7, 38.6)
- added R60: 100k, Resistor_SMD:R_0805_2012Metric_Pad1.20x1.40mm_HandSolder, F.Cu at (126.8, 110.0)
- added R61: 100k, Resistor_SMD:R_0805_2012Metric_Pad1.20x1.40mm_HandSolder, F.Cu at (125.7, 25.1)
- added R62: 220k, Resistor_SMD:R_0805_2012Metric_Pad1.20x1.40mm_HandSolder, F.Cu at (132.6, 95.2)
- added R63: 220k, Resistor_SMD:R_0805_2012Metric_Pad1.20x1.40mm_HandSolder, F.Cu at (132.6, 101.9)
- added R64: 220k, Resistor_SMD:R_0805_2012Metric_Pad1.20x1.40mm_HandSolder, F.Cu at (130.8, 38.6)
- added R65: 220k, Resistor_SMD:R_0805_2012Metric_Pad1.20x1.40mm_HandSolder, F.Cu at (130.8, 45.0)
- added R66: 220k, Resistor_SMD:R_0805_2012Metric_Pad1.20x1.40mm_HandSolder, F.Cu at (132.1, 116.6)
- added R67: 220k, Resistor_SMD:R_0805_2012Metric_Pad1.20x1.40mm_HandSolder, F.Cu at (134.6, 116.6)
- added R68: 220k, Resistor_SMD:R_0805_2012Metric_Pad1.20x1.40mm_HandSolder, F.Cu at (132.3, 25.1)
- added R69: 220k, Resistor_SMD:R_0805_2012Metric_Pad1.20x1.40mm_HandSolder, F.Cu at (136.9, 25.1)
- added R70: 220k, Resistor_SMD:R_0805_2012Metric_Pad1.20x1.40mm_HandSolder, F.Cu at (138.4, 109.2)
- added R71: 220k, Resistor_SMD:R_0805_2012Metric_Pad1.20x1.40mm_HandSolder, F.Cu at (134.1, 28.7)
- added R72: 220k, Resistor_SMD:R_0805_2012Metric_Pad1.20x1.40mm_HandSolder, F.Cu at (137.2, 116.6)
- added R73: 220k, Resistor_SMD:R_0805_2012Metric_Pad1.20x1.40mm_HandSolder, F.Cu at (134.1, 33.0)
- added R74: 1M, Resistor_SMD:R_0805_2012Metric_Pad1.20x1.40mm_HandSolder, F.Cu at (132.4, 91.9)
- added R75: 1M, Resistor_SMD:R_0805_2012Metric_Pad1.20x1.40mm_HandSolder, F.Cu at (126.7, 91.9)
- added R76: 1M, Resistor_SMD:R_0805_2012Metric_Pad1.20x1.40mm_HandSolder, F.Cu at (135.4, 39.6)
- added R77: 1M, Resistor_SMD:R_0805_2012Metric_Pad1.20x1.40mm_HandSolder, F.Cu at (135.4, 44.2)
- added R78: 220k, Resistor_SMD:R_0805_2012Metric_Pad1.20x1.40mm_HandSolder, F.Cu at (140.5, 116.1)
- added R79: 220k, Resistor_SMD:R_0805_2012Metric_Pad1.20x1.40mm_HandSolder, F.Cu at (137.4, 31.8)
- added R80: 220k, Resistor_SMD:R_0805_2012Metric_Pad1.20x1.40mm_HandSolder, F.Cu at (141.7, 112.8)
- added R81: 220k, Resistor_SMD:R_0805_2012Metric_Pad1.20x1.40mm_HandSolder, F.Cu at (138.4, 106.7)
- added R82: 220k, Resistor_SMD:R_0805_2012Metric_Pad1.20x1.40mm_HandSolder, F.Cu at (141.8, 108.3)
- added R83: 220k, Resistor_SMD:R_0805_2012Metric_Pad1.20x1.40mm_HandSolder, F.Cu at (137.4, 34.0)
- added R84: 220k, Resistor_SMD:R_0805_2012Metric_Pad1.20x1.40mm_HandSolder, F.Cu at (139.2, 44.2)
- added R85: 220k, Resistor_SMD:R_0805_2012Metric_Pad1.20x1.40mm_HandSolder, F.Cu at (139.2, 39.6)
- added R86: 1M, Resistor_SMD:R_0805_2012Metric_Pad1.20x1.40mm_HandSolder, F.Cu at (104.4, 69.8)
- added U14: INA331, Package_SO:MSOP-8_3x3mm_P0.65mm, F.Cu at (126.7, 98.7)
- added U15: INA331, Package_SO:MSOP-8_3x3mm_P0.65mm, F.Cu at (126.1, 41.7)
- added U16: INA331, Package_SO:MSOP-8_3x3mm_P0.65mm, F.Cu at (126.7, 113.5)
- added U17: INA331, Package_SO:MSOP-8_3x3mm_P0.65mm, F.Cu at (126.1, 28.5)
- added U18: OPA340NA, Package_TO_SOT_SMD:SOT-23-5, F.Cu at (138.5, 112.6)
- added U19: OPA340NA, Package_TO_SOT_SMD:SOT-23-5, F.Cu at (137.5, 28.6)
- C13, C5, C7, C8: value 4.7nF -> 470pF
- C3, C4: value 4.7nF -> 100nF
- R1, R12, R14, R15, R2, R3, R4, R6, R7, R8: value 4.99k -> 1M
- moved U8 82.8 mm to (97.0, 29.0)
- moved U1 82.0 mm to (97.0, 113.8)
- moved R5 62.0 mm to (104.8, 106.9)
- moved C13 60.4 mm to (118.6, 54.1), turned to 180 degrees
- moved U7 58.2 mm to (97.0, 42.2)
- moved R2 56.2 mm to (117.9, 85.3)
- moved U2 55.9 mm to (97.0, 99.1)
- moved R1 48.7 mm to (99.6, 62.5), turned to 90 degrees
- moved R12 40.3 mm to (99.1, 49.0), turned to 0 degrees
- moved R3 38.5 mm to (99.6, 69.8)
- moved REF** 37.2 mm to (165.1, 98.3)
- moved R15 33.4 mm to (109.2, 69.8)
- moved U6 33.3 mm to (97.0, 55.6)
- moved R4 27.7 mm to (117.9, 68.1)
- moved C5 25.1 mm to (113.5, 76.7), turned to 90 degrees
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Connections:
- C13 pad 1: GNDA -> INP6P
- C13 pad 2: Net-(C13-Pad2) -> BIASREF
- C14 pad 2: Net-(C14-Pad2) -> BIASREF
- C3 pad 2: GNDA -> Net-(C3-Pad2)
- C4 pad 1: GNDA -> Net-(C4-Pad1)
- C5 pad 1: Net-(C5-Pad1) -> Net-(C38-Pad2)
- C5 pad 2: GNDA -> Net-(C43-Pad2)
- C7 pad 1: Net-(C7-Pad1) -> Net-(C38-Pad2)
- C8 pad 2: Net-(C8-Pad2) -> Net-(C43-Pad2)
- JP3 pad 1: Net-(C14-Pad2) -> BIASREF
- R1 pad 1: Net-(C15-Pad2) -> INP4P
- R1 pad 2: Net-(JP1-Pad1) -> +5VA
- R12 pad 1: Net-(C10-Pad1) -> Net-(R12-Pad1)
- R12 pad 2: Net-(R12-Pad2) -> BIASREF
- R14 pad 1: Net-(C11-Pad1) -> Net-(C38-Pad2)
- R15 pad 1: Net-(C11-Pad2) -> Net-(C43-Pad2)
- R19 pad 2: Net-(C14-Pad2) -> BIASREF
- R2 pad 1: Net-(C1-Pad1) -> INP3P
- R2 pad 2: Net-(R2-Pad2) -> BIASREF
- R3 pad 1: Net-(C2-Pad2) -> Net-(R3-Pad1)
- R3 pad 2: Net-(R3-Pad2) -> BIASREF
- R4 pad 1: Net-(C3-Pad1) -> INP3N
- R4 pad 2: Net-(R4-Pad2) -> BIASREF
- R5 pad 1: Net-(C4-Pad2) -> GNDA
- R5 pad 2: Net-(R5-Pad2) -> Net-(R36-Pad1)
- R6 pad 1: Net-(C5-Pad1) -> INP4N
- R6 pad 2: Net-(R6-Pad2) -> +5VA
- R7 pad 1: Net-(C6-Pad2) -> INP5P
- R7 pad 2: Net-(R7-Pad2) -> +5VA
- R8 pad 1: Net-(C7-Pad1) -> INP5N
- R8 pad 2: Net-(R8-Pad2) -> +5VA
- U1 pad 1: Net-(JP1-Pad3) -> Net-(R36-Pad1)
- U1 pad 4: Net-(R2-Pad2) -> Net-(R43-Pad2)
- U1 pad 5: Net-(R3-Pad2) -> Net-(R44-Pad2)
- U2 pad 1: Net-(JP1-Pad3) -> Net-(R34-Pad1)
- U2 pad 4: Net-(R4-Pad2) -> Net-(R38-Pad2)
- U2 pad 5: Net-(R5-Pad2) -> Net-(R39-Pad2)
- U3 pad 1: Net-(JP1-Pad3) -> Net-(R3-Pad1)
- U3 pad 4: Net-(R6-Pad2) -> Net-(R14-Pad2)
- U3 pad 5: Net-(R7-Pad2) -> Net-(R15-Pad2)
- U6 pad 1: Net-(JP1-Pad3) -> Net-(R12-Pad1)
- U6 pad 4: Net-(R12-Pad2) -> Net-(C3-Pad2)
- U6 pad 5: Net-(R13-Pad2) -> Net-(C4-Pad2)
- U7 pad 1: Net-(JP1-Pad3) -> Net-(R35-Pad1)
- U7 pad 4: Net-(R14-Pad2) -> Net-(R40-Pad2)
- U7 pad 5: Net-(R15-Pad2) -> Net-(R41-Pad2)
- U9 pad 1: Net-(C1-Pad1) -> INP8N
- U9 pad 10: Net-(C9-Pad2) -> INP4P
- U9 pad 11: Net-(C10-Pad1) -> INP3N
- U9 pad 12: Net-(C10-Pad2) -> INP3P
- U9 pad 13: Net-(C11-Pad1) -> INP2N
- U9 pad 14: Net-(C11-Pad2) -> INP2P
- U9 pad 15: Net-(C12-Pad1) -> INP1N
- U9 pad 16: Net-(C13-Pad2) -> INP1P
- U9 pad 17: Net-(C15-Pad2) -> GNDA
- U9 pad 2: Net-(C2-Pad2) -> INP8P
- U9 pad 3: Net-(C3-Pad1) -> INP7N
- U9 pad 4: Net-(C4-Pad2) -> INP7P
- U9 pad 5: Net-(C5-Pad1) -> INP6N
- U9 pad 6: Net-(C6-Pad2) -> INP6P
- U9 pad 63: Net-(C14-Pad2) -> BIASREF
- U9 pad 7: Net-(C7-Pad1) -> INP5N
- U9 pad 8: Net-(C8-Pad2) -> INP5P
- U9 pad 9: Net-(C9-Pad1) -> INP4N
Routing:
- net BIASREF: track 0.00 -> 612.8 mm
- net +5VA: track 102.2 -> 334.0 mm, vias 1 -> 6
- net Net-(JP1-Pad3): track 177.0 -> 0.00 mm
- net INP1P: track 0.00 -> 68.9 mm
- net INP8P: track 0.00 -> 59.5 mm
- net INP1N: track 0.00 -> 57.7 mm
- net Net-(C14-Pad2): track 56.1 -> 0.00 mm
- net Net-(C13-Pad2): track 52.7 -> 0.00 mm
- net Net-(C1-Pad1): track 52.6 -> 0.00 mm
- net Net-(R37-Pad1): track 52.8 -> 6.47 mm
- net Net-(C2-Pad2): track 45.6 -> 0.00 mm
- net Net-(C12-Pad1): track 44.7 -> 0.00 mm
- net INP2P: track 0.00 -> 44.1 mm
- net INP7P: track 0.00 -> 42.2 mm
- net INP8N: track 0.00 -> 41.4 mm
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Other:
- board text added: "EMG-8[6]x Rev.3"
- board text removed: "Bias"
- board text removed: "BiasIn"
- board text removed: "EMG-8x Rev.2"
- board text removed: "GNDA"
- board text removed: "IN1"
- board text removed: "IN2"
- board text removed: "IN3"
- board text removed: "IN4"
- board text removed: "IN5"
- board text removed: "IN6"
- board text removed: "IN7"
- board text removed: "IN8"
- board text removed: "SRB1"

Commit message: working copy
Parts:
- removed C3, C43, C62, C63: 100nF, Capacitor_SMD:C_0805_2012Metric_Pad1.18x1.45mm_HandSolder
- removed R31, R70, R71, R72, R73, R78, R79, R80, R83: 220k, Resistor_SMD:R_0805_2012Metric_Pad1.20x1.40mm_HandSolder
- removed R49, R51, R86: 1M, Resistor_SMD:R_0805_2012Metric_Pad1.20x1.40mm_HandSolder
- removed U18, U19: OPA340NA, Package_TO_SOT_SMD:SOT-23-5
- added D1: LED, LED_SMD:LED_0805_2012Metric, F.Cu at (176.0, 32.9)
- added D2: LED, LED_SMD:LED_0805_2012Metric, F.Cu at (172.4, 32.9)
- added D3: LED, LED_SMD:LED_0805_2012Metric, F.Cu at (168.7, 32.9)
- added R10: 10k, Resistor_SMD:R_0805_2012Metric_Pad1.20x1.40mm_HandSolder, F.Cu at (115.6, 54.2)
- added R11: 10k, Resistor_SMD:R_0805_2012Metric_Pad1.20x1.40mm_HandSolder, F.Cu at (114.6, 62.2)
- added R13: 300, Resistor_SMD:R_0805_2012Metric_Pad1.20x1.40mm_HandSolder, F.Cu at (176.0, 37.4)
- added R16: 300, Resistor_SMD:R_0805_2012Metric_Pad1.20x1.40mm_HandSolder, F.Cu at (172.4, 37.4)
- added R17: 300, Resistor_SMD:R_0805_2012Metric_Pad1.20x1.40mm_HandSolder, F.Cu at (168.7, 37.4)
- added R9: 100k, Resistor_SMD:R_0805_2012Metric_Pad1.20x1.40mm_HandSolder, F.Cu at (110.5, 72.7)
- added U4: INA331, Package_SO:MSOP-8_3x3mm_P0.65mm, F.Cu at (104.8, 72.7)
- added U5: INA331, Package_SO:MSOP-8_3x3mm_P0.65mm, F.Cu at (104.7, 51.3)
- C13, C37, C5, C64: value 470pF -> 0.1uF
- C38, C4, C58, C59, C60, C61: value 100nF -> 22uF
- C46, C47: value 4.7nF -> 0.1u
- C48, C49, C50, C51, C52, C53, C54, C55, C56, C57: value 4.7nF -> 0.1uF
- C7, C8: value 470pF -> 0.068uF
- R1, R4, R6, R7, R8: value 1M -> 10k
- R12, R14, R15, R3, R45, R53, R75, R77: value 1M -> 5.1k
- R2, R74, R76: value 1M -> 100k
- R24, R25, R62, R64, R66, R82, R85: value 220k -> 100k
- R28, R29, R84: value 220k -> 5.1k
- R30, R63, R65, R67, R69, R81: value 220k -> 10k
- R35, R36, R37, R38, R39, R40, R41, R43, R44, R46, R47, R5: value 4.99k -> 5.1k
- moved REF** 66.6 mm to (164.8, 102.7)
- moved R6 30.5 mm to (116.2, 89.9), turned to 180 degrees
- moved R1 29.9 mm to (116.2, 87.4), turned to 180 degrees
- moved REF** 24.2 mm to (141.0, 101.0)
- moved C64 24.2 mm to (98.3, 51.2), turned to 90 degrees
- moved R8 23.3 mm to (116.2, 84.8), turned to 180 degrees
- moved R7 22.1 mm to (116.2, 82.3), turned to 180 degrees
- moved R2 21.3 mm to (104.2, 69.1), turned to 0 degrees
- moved C13 17.5 mm to (101.2, 55.9), turned to 270 degrees
- moved C5 15.5 mm to (98.6, 72.6)
- moved R28 15.1 mm to (104.1, 55.9), turned to 90 degrees
- moved R84 13.4 mm to (139.2, 30.8), turned to 270 degrees
- moved R25 13.0 mm to (104.5, 48.3), turned to 180 degrees
- moved C7 12.5 mm to (101.9, 77.4)
- moved R29 12.2 mm to (106.9, 55.9), turned to 90 degrees
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Connections:
- C13 pad 1: INP6P -> Net-(C13-Pad1)
- C13 pad 2: BIASREF -> GNDA
- C37 pad 1: BIASREF -> GNDA
- C37 pad 2: INP6N -> Net-(C37-Pad2)
- C38 pad 1: INP3P -> INP5P
- C4 pad 2: Net-(C4-Pad2) -> INP6P
- C48 pad 2: BIASREF -> GNDA
- C49 pad 1: BIASREF -> GNDA
- C5 pad 1: Net-(C38-Pad2) -> Net-(C5-Pad1)
- C52 pad 2: BIASREF -> GNDA
- C53 pad 1: BIASREF -> GNDA
- C60 pad 1: Net-(C60-Pad1) -> INP1P
- C61 pad 1: Net-(C61-Pad1) -> INP8P
- C64 pad 1: INP6P -> Net-(C13-Pad1)
- C64 pad 2: INP6N -> Net-(C37-Pad2)
- C7 pad 1: Net-(C38-Pad2) -> Net-(C5-Pad1)
- R1 pad 1: INP4P -> INP3N
- R14 pad 1: Net-(C38-Pad2) -> Net-(C5-Pad1)
- R2 pad 1: INP3P -> Net-(R2-Pad1)
- R2 pad 2: BIASREF -> Net-(R2-Pad2)
- R24 pad 1: BIASREF -> Net-(R24-Pad1)
- R24 pad 2: Net-(C3-Pad1) -> Net-(C4-Pad1)
- R25 pad 1: Net-(C4-Pad1) -> Net-(R25-Pad1)
- R25 pad 2: BIASREF -> Net-(R24-Pad1)
- R28 pad 1: Net-(C3-Pad1) -> Net-(R28-Pad1)
- R28 pad 2: INP6P -> Net-(C13-Pad1)
- R29 pad 1: Net-(C4-Pad1) -> Net-(R29-Pad1)
- R29 pad 2: INP6N -> Net-(C37-Pad2)
- R30 pad 2: INP3P -> INP5P
- R4 pad 1: INP3N -> BIASREF
- R4 pad 2: BIASREF -> INP5N
- R6 pad 1: INP4N -> INP3P
- R66 pad 1: Net-(C62-Pad1) -> INP1P
- R67 pad 2: Net-(C62-Pad1) -> INP1P
- R68 pad 1: Net-(C63-Pad1) -> INP8P
- R69 pad 2: Net-(C63-Pad1) -> INP8P
- R7 pad 1: INP5P -> INP4N
- R76 pad 1: GNDA -> INP7N
- R76 pad 2: INP7N -> GNDA
- R8 pad 1: INP5N -> INP4P
- U14 pad 8: GNDA -> +5VA
- U15 pad 8: GNDA -> +5VA
- U16 pad 8: GNDA -> +5VA
- U17 pad 8: GNDA -> +5VA
- U6 pad 4: Net-(C3-Pad2) -> Net-(R28-Pad1)
- U6 pad 5: Net-(C4-Pad2) -> Net-(R29-Pad1)
Routing:
- net BIASREF: track 612.8 -> 460.7 mm
- net Net-(R17-Pad2): track 0.00 -> 40.0 mm
- net Net-(R16-Pad2): track 0.00 -> 34.5 mm
- net Net-(R13-Pad2): track 0.00 -> 29.1 mm
- net +5VA: track 334.0 -> 349.2 mm, vias 6 -> 7
- net Net-(C3-Pad2): track 15.0 -> 0.00 mm
- net Net-(R2-Pad1): track 0.00 -> 14.4 mm
- net Net-(C37-Pad2): track 0.00 -> 14.3 mm
- net Net-(R24-Pad1): track 0.00 -> 12.3 mm
- net Net-(C13-Pad1): track 0.00 -> 11.8 mm
- net Net-(C4-Pad2): track 11.7 -> 0.00 mm
- net INP4P: track 35.9 -> 24.5 mm
- net INP8N: track 41.4 -> 52.7 mm
- net Net-(C5-Pad1): track 0.00 -> 10.7 mm
- net INP4N: track 32.4 -> 22.5 mm
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Other:
- board text added: "EMG-8[6]x Rev.4"
- board text added: "MIREA(MGUPI) KB2(KB3)"
- board text added: "Rf-Lab.org (2021)"
- board text added: "U5"
- board text removed: "EMG-8[6]x Rev.3"
- board text removed: "MGUPI/MIREA/KB3/KB2"
- board text removed: "Rf-Lab.org"

Commit message: Revision 4
Parts:
- added C1: 0.1uF, Capacitor_SMD:C_0805_2012Metric_Pad1.18x1.45mm_HandSolder, F.Cu at (129.2, 24.8)
- added C10: 0.1uF, Capacitor_SMD:C_0805_2012Metric_Pad1.18x1.45mm_HandSolder, F.Cu at (132.8, 112.8)
- added C2: 0.1uF, Capacitor_SMD:C_0805_2012Metric_Pad1.18x1.45mm_HandSolder, F.Cu at (127.1, 37.2)
- added C3: 0.1uF, Capacitor_SMD:C_0805_2012Metric_Pad1.18x1.45mm_HandSolder, F.Cu at (108.5, 48.1)
- added C6: 0.1uF, Capacitor_SMD:C_0805_2012Metric_Pad1.18x1.45mm_HandSolder, F.Cu at (132.8, 97.8)
- added C9: 0.1uF, Capacitor_SMD:C_0805_2012Metric_Pad1.18x1.45mm_HandSolder, F.Cu at (107.8, 69.1)
- moved REF** 38.4 mm to (123.0, 67.1), turned to 90 degrees
- moved C58 1.95 mm to (132.8, 100.2)
- moved R66 1.48 mm to (132.7, 110.2)
- moved R25 1.15 mm to (103.4, 48.1)
- moved C60 1.11 mm to (132.8, 115.5)
- moved R81 1.09 mm to (132.7, 107.6)
- moved R68 1.02 mm to (133.1, 25.4)
- moved R67 0.98 mm to (132.7, 118.1)
- moved R63 0.82 mm to (132.7, 102.7)
- moved R64 0.63 mm to (130.2, 38.6)
- moved R2 0.57 mm to (103.6, 69.1)
- moved R24 0.45 mm to (110.2, 51.6)
- moved R74 0.45 mm to (132.7, 92.2)
- moved C20 0.40 mm to (144.1, 83.6)
- moved C21 0.33 mm to (147.0, 84.0)
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Routing:
- net +5VA: track 349.2 -> 357.0 mm
- net INP2P: track 46.8 -> 52.5 mm
- net INP1P: track 68.1 -> 72.9 mm
- net Net-(R24-Pad1): track 12.3 -> 16.5 mm
- net BIASREF: track 460.7 -> 463.0 mm
- net GNDA: track 28.2 -> 29.9 mm, vias 23 -> 24
- net INP1N: track 56.1 -> 56.8 mm
- net Net-(R2-Pad1): track 14.4 -> 15.1 mm
- net Net-(C58-Pad2): track 8.08 -> 8.60 mm
- net GNDD: vias 6 -> 9

Commit message: schematic verification
Parts:
- C14: value 1n5 -> 0.01uF
- R19: value 1M -> 390k
