File: hw_platform/ADS1299EMG8xR2/ADS1299EMG8xR2.sch (KiCad schematic (older format))
At the start: 83 parts

Commit message: all footprints completed
Parts:
- removed C?: 1u, symbol Device:C
- removed C?: 0.1u, symbol Device:C
- BT1, BT2: renamed from BT?; footprint (none) -> Battery:BatteryHolder_Blossom_1x18650
- C1, C10, C11, C12, C13, C14, C15, C16, C17, C19, C2, C20, C22, C23, C27, C28, C29, C3, C31, C32, C33, C34, C36, C39, C4, C40, C41, C42, C5, C6, C7, C8, C9: renamed from C?; footprint (none) -> Capacitor_SMD:C_0805_2012Metric_Pad1.18x1.45mm_HandSolder
- C18, C24, C25, C26, C30, C35: renamed from C?; value CP1 -> 10uF; footprint (none) -> Capacitor_Tantalum_SMD:CP_EIA-3528-21_Kemet-B_Pad1.50x2.35mm_HandSolder
- C21: renamed from C?; footprint (none) -> Capacitor_SMD:C_1206_3216Metric_Pad1.33x1.80mm_HandSolder
- JP1, JP2, JP4, JP6: renamed from JP?; footprint (none) -> Jumper:SolderJumper-3_P1.3mm_Bridged2Bar12_Pad1.0x1.5mm_NumberLabels
- JP3, JP5: renamed from JP?; footprint (none) -> Jumper:SolderJumper-2_P1.3mm_Bridged2Bar_Pad1.0x1.5mm
- R1, R10, R11, R12, R13, R14, R15, R16, R17, R18, R19, R2, R20, R3, R4, R5, R6, R7, R8, R9: renamed from R?; footprint (none) -> Resistor_SMD:R_0805_2012Metric_Pad1.20x1.40mm_HandSolder
- U1, U2, U3, U4, U5, U6, U7, U8: renamed from U?; footprint (none) -> Connector_Audio:Jack_3.5mm_PJ-325-P5
- U10, U11, U12: renamed from U?; footprint (none) -> Package_TO_SOT_SMD:TO-252-3_TabPin2
- U13: renamed from U?; footprint (none) -> Package_DIP:DIP-38_W22.86m_P2.54mm_ESP32_DevKitC
- U9: renamed from U?; footprint (none) -> Package_QFP:PQFP-64-12x12mm_P0.5_ADS1299

Commit message: partial routed
Parts:
- JP1, JP2, JP4, JP6: footprint Jumper:SolderJumper-3_P1.3mm_Bridged2Bar12_Pad1.0x1.5mm_NumberLabels -> Connector_PinHeader_2.54mm:PinHeader_1x03_P2.54mm_Vertical
- JP3, JP5: footprint Jumper:SolderJumper-2_P1.3mm_Bridged2Bar_Pad1.0x1.5mm -> Connector_PinHeader_2.54mm:PinHeader_1x02_P2.54mm_Vertical
Changed lines of the file:
@@
 F 0 "JP2" H 1050 1154 50  0000 C CNN
 F 1 "Jumper_3_Bridged12" H 1050 1063 50  0000 C CNN
-F 2 "Jumper:SolderJumper-3_P1.3mm_Bridged2Bar12_Pad1.0x1.5mm_NumberLabels" H 1050 950 50  0001 C CNN
+F 2 "Connector_PinHeader_2.54mm:PinHeader_1x03_P2.54mm_Vertical" H 1050 950 50  0001 C CNN
 F 3 "~" H 1050 950 50  0001 C CNN
 	1    1050 950
@@
 F 0 "JP1" H 750 7254 50  0000 C CNN
 F 1 "Jumper_3_Bridged12" H 750 7163 50  0000 C CNN
-F 2 "Jumper:SolderJumper-3_P1.3mm_Bridged2Bar12_Pad1.0x1.5mm_NumberLabels" H 750 7050 50  0001 C CNN
+F 2 "Connector_PinHeader_2.54mm:PinHeader_1x03_P2.54mm_Vertical" H 750 7050 50  0001 C CNN
 F 3 "~" H 750 7050 50  0001 C CNN
 	1    750  7050
@@
 F 0 "JP3" H 3650 1350 50  0000 C CNN
 F 1 "Jumper" H 4050 1350 50  0000 C CNN
-F 2 "Jumper:SolderJumper-2_P1.3mm_Bridged2Bar_Pad1.0x1.5mm" H 3850 1200 50  0001 C CNN
+F 2 "Connector_PinHeader_2.54mm:PinHeader_1x02_P2.54mm_Vertical" H 3850 1200 50  0001 C CNN
 F 3 "~" H 3850 1200 50  0001 C CNN
 	1    3850 1200
@@
 F 0 "JP4" H 6000 5754 50  0000 C CNN
 F 1 "Jumper_3_Bridged12" H 6000 5663 50  0000 C CNN
-F 2 "Jumper:SolderJumper-3_P1.3mm_Bridged2Bar12_Pad1.0x1.5mm_NumberLabels" H 6000 5550 50  0001 C CNN
+F 2 "Connector_PinHeader_2.54mm:PinHeader_1x03_P2.54mm_Vertical" H 6000 5550 50  0001 C CNN
 F 3 "~" H 6000 5550 50  0001 C CNN
 	1    6000 5550
@@
 F 0 "JP6" H 9400 5754 50  0000 C CNN
 F 1 "Jumper_3_Bridged12" H 9400 5663 50  0000 C CNN
-F 2 "Jumper:SolderJumper-3_P1.3mm_Bridged2Bar12_Pad1.0x1.5mm_NumberLabels" H 9400 5550 50  0001 C CNN
+F 2 "Connector_PinHeader_2.54mm:PinHeader_1x03_P2.54mm_Vertical" H 9400 5550 50  0001 C CNN
 F 3 "~" H 9400 5550 50  0001 C CNN
 	1    9400 5550
@@
 F 0 "JP5" H 6050 7114 50  0000 C CNN
 F 1 "Jumper" H 6050 7023 50  0000 C CNN
-F 2 "Jumper:SolderJumper-2_P1.3mm_Bridged2Bar_Pad1.0x1.5mm" H 6050 6850 50  0001 C CNN
+F 2 "Connector_PinHeader_2.54mm:PinHeader_1x02_P2.54mm_Vertical" H 6050 6850 50  0001 C CNN
 F 3 "~" H 6050 6850 50  0001 C CNN
 	1    6050 6850

Commit message: REvision2_release
Parts:
- added R21, R22: 10k, Resistor_SMD:R_0805_2012Metric_Pad1.20x1.40mm_HandSolder, symbol Device:R
Connections:
- net GNDA: now also U9.18 (SRB2), U9.60 (BIASREF)
- net GNDD: now also R21.1, R22.1
- net ADS_GPIO1: no longer names the net of U9.42 (GPIO1)
- net ADS_GPIO1: now also R22.2; no longer U13.10 (gpio26)
- net ADS_GPIO2: no longer names the net of U9.44 (GPIO2)
- net ADS_GPIO2: now also R21.2; no longer U13.11 (gpio27)
Changed lines of the file:
@@
 L power:GNDD #PWR031
 U 1 1 5F8C9FFB
-P 6150 3750
-F 0 "#PWR031" H 6150 3500 50  0001 C CNN
-F 1 "GNDD" V 6150 3550 50  0000 C CNN
-F 2 "" H 6150 3750 50  0001 C CNN
-F 3 "" H 6150 3750 50  0001 C CNN
-	1    6150 3750
+P 6450 3650
+F 0 "#PWR031" H 6450 3400 50  0001 C CNN
+F 1 "GNDD" V 6450 3450 50  0000 C CNN
+F 2 "" H 6450 3650 50  0001 C CNN
+F 3 "" H 6450 3650 50  0001 C CNN
+	1    6450 3650
 	0    -1   -1   0
 $EndComp
-Wire Wire Line
-	5950 3750 6150 3750
 Wire Wire Line
 	5950 4050 7000 4050
@@
 Wire Wire Line
 	9600 3400 9700 3400
-Text GLabel 5950 3450 2    50   Input ~ 0
-ADS_GPIO2
-Text GLabel 9600 3700 2    50   Input ~ 0
-ADS_GPIO2
-Text GLabel 5950 3650 2    50   Input ~ 0
-ADS_GPIO1
-Text GLabel 9600 3800 2    50   Input ~ 0
-ADS_GPIO1
 $Comp
 L Regulator_Linear:LM1117-3.3 U11
@@
 Text Notes 5900 7000 0    50   ~ 0
 Battery
+$Comp
+L Device:R R21
+U 1 1 5FA1F136
+P 6200 3450
+F 0 "R21" V 6150 3650 50  0000 C CNN
+F 1 "10k" V 6200 3450 50  0000 C CNN
+F 2 "Resistor_SMD:R_0805_2012Metric_Pad1.20x1.40mm_HandSolder" V 6130 3450 50  0001 C CNN
+F 3 "~" H 6200 3450 50  0001 C CNN
+	1    6200 3450
+	0    1    1    0
+$EndComp
+Wire Wire Line
+	5950 3450 6050 3450
+$Comp
+L power:GNDD #PWR055
+U 1 1 5FA39E6B
+P 6450 3450
+F 0 "#PWR055" H 6450 3200 50  0001 C CNN
+F 1 "GNDD" V 6450 3250 50  0000 C CNN
+F 2 "" H 6450 3450 50  0001 C CNN
+F 3 "" H 6450 3450 50  0001 C CNN
+	1    6450 3450
+	0    -1   -1   0
+$EndComp
+Wire Wire Line
+	6350 3450 6450 3450
+$Comp
+L Device:R R22
+U 1 1 5FA53C02
+P 6200 3650
+F 0 "R22" V 6150 3850 50  0000 C CNN
+F 1 "10k" V 6200 3650 50  0000 C CNN
+F 2 "Resistor_SMD:R_0805_2012Metric_Pad1.20x1.40mm_HandSolder" V 6130 3650 50  0001 C CNN
+F 3 "~" H 6200 3650 50  0001 C CNN
+	1    6200 3650
+	0    1    1    0
+$EndComp
+Wire Wire Line
+	5950 3750 6400 3750
+Wire Wire Line
+	6400 3750 6400 3650
+Wire Wire Line
+	6400 3650 6450 3650
+Wire Wire Line
+	6350 3650 6400 3650
+Connection ~ 6400 3650
+Wire Wire Line
+	5950 3650 6050 3650
+$Comp
+L power:GNDA #PWR0101
+U 1 1 5FAD31ED
+P 4150 5000
+F 0 "#PWR0101" H 4150 4750 50  0001 C CNN
+F 1 "GNDA" H 4155 4827 50  0000 C CNN
+F 2 "" H 4150 5000 50  0001 C CNN
+F 3 "" H 4150 5000 50  0001 C CNN
+	1    4150 5000
+	1    0    0    -1
+$EndComp
+Wire Wire Line
+	4150 4900 4150 5000
+$Comp
+L power:GNDA #PWR0102
+U 1 1 5FAF39E8
+P 4450 2550
+F 0 "#PWR0102" H 4450 2300 50  0001 C CNN
+F 1 "GNDA" H 4455 2377 50  0000 C CNN
+F 2 "" H 4450 2550 50  0001 C CNN
+F 3 "" H 4450 2550 50  0001 C CNN
+	1    4450 2550
+	-1   0    0    1
+$EndComp
+Wire Wire Line
+	4450 2550 4450 2650
 $EndSCHEMATC

Commit message: revision 3
Parts:
- removed C1, C10, C11, C12, C13, C15, C2, C3, C4, C5, C6, C7, C8, C9: 4.7nF, Capacitor_SMD:C_0805_2012Metric_Pad1.18x1.45mm_HandSolder, symbol Device:C
- removed JP1, JP2: Jumper_3_Bridged12, Connector_PinHeader_2.54mm:PinHeader_1x03_P2.54mm_Vertical, symbol Jumper:Jumper_3_Bridged12
- removed R1, R10, R11, R12, R13, R14, R15, R16, R17, R18, R2, R3, R4, R5, R6, R7, R8, R9: 4.99k, Resistor_SMD:R_0805_2012Metric_Pad1.20x1.40mm_HandSolder, symbol Device:R
- removed U1, U2, U3, U4, U5, U6, U7, U8: PJ-325-5P, Connector_Audio:Jack_3.5mm_PJ-325-P5, symbol Connector:PJ-325-5P
Connections:
- net GNDA: now also U9.17 (SRB1)
- net INP8N: now reaches U9.1 (IN8N)
- net INP4P: now reaches U9.10 (IN4P)
- net INP3N: now reaches U9.11 (IN3N)
- net INP3P: now reaches U9.12 (IN3P)
- net INP2N: now reaches U9.13 (IN2N)
- net INP2P: now reaches U9.14 (IN2P)
- net INP1N: now reaches U9.15 (IN1N)
- net INP1P: now reaches U9.16 (IN1P)
- net INP8P: now reaches U9.2 (IN8P)
- net INP7N: now reaches U9.3 (IN7N)
- net INP7P: now reaches U9.4 (IN7P)
- net INP6N: now reaches U9.5 (IN6N)
- net INP6P: now reaches U9.6 (IN6P)
- net BIASREF: now reaches C14.2, JP3.1, R19.2, U9.63 (BIASOUT)
- net INP5N: now reaches U9.7 (IN5N)
- net INP5P: now reaches U9.8 (IN5P)
- net INP4N: now reaches U9.9 (IN4N)
- no-connect marks 16 -> 0
Other:
- moved on the sheet: BT1, BT2, C27, C28, C29, C31, C32, C33, C34, C36, R20

Commit message: working copy
Parts:
- added D1, D2, D3: LED, LED_SMD:LED_0805_2012Metric, symbol Device:LED
- added R13, R16, R17: 300, Resistor_SMD:R_0805_2012Metric_Pad1.20x1.40mm_HandSolder, symbol Device:R
Connections:
- net GNDD: now also D1.1 (K), D2.1 (K), D3.1 (K)
- net at U13.10 (gpio26): now also R16.2
- net at U13.11 (gpio27): now also R13.2
- net at U13.9 (gpio25): now also R17.2
- new net: D1.2 (A), R13.1
- new net: D2.2 (A), R16.1
- new net: D3.2 (A), R17.1
Changed lines of the file:
@@
 Sheet 1 2
 Title "EMG8x"
-Date "2021-01-06"
-Rev "R3"
+Date "2021-03-15"
+Rev "R4"
 Comp "RF-LAB.ORG/KB-3/KB-2/MGUPI/MIREA"
-Comment1 "active passband (2 types)"
-Comment2 "Four types analogue filters: passive passband (2 types)"
-Comment3 "Based on ADS1299, WiFi/BLE based on ESP32"
-Comment4 "8 channel EMG hardware platform"
+Comment1 "ESP32 (2Cores x 250MHz +WiFi+ BLE)"
+Comment2 "Four identical interfaces based on INA331 amplifier"
+Comment3 "Based on 8 channel ADC ADS1299 (4 channel switched off for R4)"
+Comment4 "4 channel wireless EMG acquisition platform"
 $EndDescr
 $Comp
@@
 	2550 1600 3250 1600
 $Sheet
-S 1150 1450 500  150
+S 900  1550 800  450
 U 5FF7A86A
-F0 "iamp" 50
+F0 "Analogue interfaces" 50
 F1 "iamp.sch" 50
 $EndSheet
@@
 Wire Wire Line
 	4050 4900 4050 5000
+$Comp
+L Device:R R13
+U 1 1 60AB8BF3
+P 10350 3700
+F 0 "R13" V 10300 3500 50  0000 C CNN
+F 1 "300" V 10350 3700 50  0000 C CNN
+F 2 "Resistor_SMD:R_0805_2012Metric_Pad1.20x1.40mm_HandSolder" V 10280 3700 50  0001 C CNN
+F 3 "~" H 10350 3700 50  0001 C CNN
+	1    10350 3700
+	0    1    1    0
+$EndComp
+$Comp
+L Device:R R16
+U 1 1 60ABA011
+P 10350 3800
+F 0 "R16" V 10300 3600 50  0000 C CNN
+F 1 "300" V 10350 3800 50  0000 C CNN
+F 2 "Resistor_SMD:R_0805_2012Metric_Pad1.20x1.40mm_HandSolder" V 10280 3800 50  0001 C CNN
+F 3 "~" H 10350 3800 50  0001 C CNN
+	1    10350 3800
+	0    1    1    0
+$EndComp
+$Comp
+L Device:R R17
+U 1 1 60ABA181
+P 10350 3900
+F 0 "R17" V 10300 3700 50  0000 C CNN
+F 1 "300" V 10350 3900 50  0000 C CNN
+F 2 "Resistor_SMD:R_0805_2012Metric_Pad1.20x1.40mm_HandSolder" V 10280 3900 50  0001 C CNN
+F 3 "~" H 10350 3900 50  0001 C CNN
+	1    10350 3900
+	0    1    1    0
+$EndComp
+Wire Wire Line
+	9600 3700 10200 3700
+Wire Wire Line
+	9600 3800 10200 3800
+Wire Wire Line
+	9600 3900 10200 3900
+$Comp
+L Device:LED D1
+U 1 1 60AEA16B
+P 10600 3350
+F 0 "D1" H 10700 3300 50  0000 C CNN
+F 1 "LED" H 10850 3300 50  0000 C CNN
+F 2 "LED_SMD:LED_0805_2012Metric" H 10600 3350 50  0001 C CNN
+F 3 "~" H 10600 3350 50  0001 C CNN
+	1    10600 3350
+	0    1    1    0
+$EndComp
+$Comp
+L Device:LED D2
+U 1 1 60AEAE4C
+P 10800 3350
+F 0 "D2" H 10900 3300 50  0000 C CNN
+F 1 "LED" H 11050 3300 50  0000 C CNN
+F 2 "LED_SMD:LED_0805_2012Metric" H 10800 3350 50  0001 C CNN
+F 3 "~" H 10800 3350 50  0001 C CNN
+	1    10800 3350
+	0    1    1    0
+$EndComp
+$Comp
+L Device:LED D3
+U 1 1 60AEB100
+P 11000 3350
+F 0 "D3" H 11100 3300 50  0000 C CNN
+F 1 "LED" H 11250 3300 50  0000 C CNN
+F 2 "LED_SMD:LED_0805_2012Metric" H 11000 3350 50  0001 C CNN
+F 3 "~" H 11000 3350 50  0001 C CNN
+	1    11000 3350
+	0    1    1    0
+$EndComp
+Wire Wire Line
+	10500 3700 10600 3700
+Wire Wire Line
+	10500 3800 10800 3800
+Wire Wire Line
+	10500 3900 11000 3900
+$Comp
+L power:GNDD #PWR0117
+U 1 1 60B4C9D6
+P 10600 2900
+F 0 "#PWR0117" H 10600 2650 50  0001 C CNN
+F 1 "GNDD" H 10600 2750 50  0000 C CNN
+F 2 "" H 10600 2900 50  0001 C CNN
+F 3 "" H 10600 2900 50  0001 C CNN
+	1    10600 2900
+	-1   0    0    1
+$EndComp
+Wire Wire Line
+	10600 3200 10600 3000
+Wire Wire Line
+	10800 3200 10800 3000
+Wire Wire Line
+	10800 3000 10600 3000
+Connection ~ 10600 3000
+Wire Wire Line
+	10600 3000 10600 2900
+Wire Wire Line
+	11000 3200 11000 3000
+Wire Wire Line
+	11000 3000 10800 3000
+Connection ~ 10800 3000
+Wire Wire Line
+	10600 3700 10600 3500
+Wire Wire Line
+	10800 3800 10800 3500
+Wire Wire Line
+	11000 3900 11000 3500
 $EndSCHEMATC

Commit message: Revision 4
Other:
- moved on the sheet: BT1, BT2
Changed lines of the file:
@@
 Date "2021-03-15"
 Rev "R4"
-Comp "RF-LAB.ORG/KB-3/KB-2/MGUPI/MIREA"
-Comment1 "ESP32 (2Cores x 250MHz +WiFi+ BLE)"
-Comment2 "Four identical interfaces based on INA331 amplifier"
-Comment3 "Based on 8 channel ADC ADS1299 (4 channel switched off for R4)"
-Comment4 "4 channel wireless EMG acquisition platform"
+Comp "RF-LAB.ORG, MIREA.RU KB2 (KB3)"
+Comment1 "Built on ESP32 SOC (2Cores x 250MHz +WiFi+ BLE)"
+Comment2 "Six identical analogue interfaces with INA331 amplifier"
+Comment3 "Based on 8 channel ADC ADS1299 (2 channel switched off for R4)"
+Comment4 "Wireless EMG acquisition platform"
 $EndDescr
 $Comp
@@
 L Device:Battery_Cell BT1
 U 1 1 5FBDEC7D
-P 5150 1100
-F 0 "BT1" H 5268 1196 50  0000 L CNN
-F 1 "Battery_Cell" H 5268 1105 50  0000 L CNN
-F 2 "Battery:BatteryHolder_Blossom_1x18650" V 5150 1160 50  0001 C CNN
-F 3 "~" V 5150 1160 50  0001 C CNN
-	1    5150 1100
+P 8650 2200
+F 0 "BT1" H 8768 2296 50  0000 L CNN
+F 1 "Battery_Cell" H 8768 2205 50  0000 L CNN
+F 2 "Battery:BatteryHolder_Blossom_1x18650" V 8650 2260 50  0001 C CNN
+F 3 "~" V 8650 2260 50  0001 C CNN
+	1    8650 2200
 	0    -1   -1   0
 $EndComp
@@
 L Device:Battery_Cell BT2
 U 1 1 5FBE0428
-P 5650 1100
-F 0 "BT2" H 5768 1196 50  0000 L CNN
-F 1 "Battery_Cell" H 5768 1105 50  0000 L CNN
-F 2 "Battery:BatteryHolder_Blossom_1x18650" V 5650 1160 50  0001 C CNN
-F 3 "~" V 5650 1160 50  0001 C CNN
-	1    5650 1100
+P 9150 2200
+F 0 "BT2" H 9268 2296 50  0000 L CNN
+F 1 "Battery_Cell" H 9268 2205 50  0000 L CNN
+F 2 "Battery:BatteryHolder_Blossom_1x18650" V 9150 2260 50  0001 C CNN
+F 3 "~" V 9150 2260 50  0001 C CNN
+	1    9150 2200
 	0    -1   -1   0
 $EndComp
@@
 L power:GNDD #PWR051
 U 1 1 5FBE0CC7
-P 5900 1100
-F 0 "#PWR051" H 5900 850 50  0001 C CNN
-F 1 "GNDD" V 5900 900 50  0000 C CNN
-F 2 "" H 5900 1100 50  0001 C CNN
-F 3 "" H 5900 1100 50  0001 C CNN
-	1    5900 1100
+P 9400 2200
+F 0 "#PWR051" H 9400 1950 50  0001 C CNN
+F 1 "GNDD" V 9400 2000 50  0000 C CNN
+F 2 "" H 9400 2200 50  0001 C CNN
+F 3 "" H 9400 2200 50  0001 C CNN
+	1    9400 2200
 	0    -1   -1   0
 $EndComp
@@
 L power:+6V #PWR042
 U 1 1 5FBE119E
-P 4800 1100
-F 0 "#PWR042" H 4800 950 50  0001 C CNN
-F 1 "+6V" V 4800 1200 50  0000 L CNN
-F 2 "" H 4800 1100 50  0001 C CNN
-F 3 "" H 4800 1100 50  0001 C CNN
-	1    4800 1100
+P 8300 2200
+F 0 "#PWR042" H 8300 2050 50  0001 C CNN
+F 1 "+6V" V 8300 2300 50  0000 L CNN
+F 2 "" H 8300 2200 50  0001 C CNN
+F 3 "" H 8300 2200 50  0001 C CNN
+	1    8300 2200
 	0    -1   -1   0
 $EndComp
 Wire Wire Line
-	4800 1100 4950 1100
-Wire Wire Line
-	5250 1100 5450 1100
-Wire Wire Line
-	5750 1100 5900 1100
+	8300 2200 8450 2200
+Wire Wire Line
+	8750 2200 8950 2200
+Wire Wire Line
+	9250 2200 9400 2200
 $Comp
 L Device:R R20

Commit message: schematic verification
Parts:
- C14: value 1n5 -> 0.01uF
- R19: value 1M -> 390k
- U13: symbol MCU_Espressif:ESP32-DevKitC -> ADS1299EMG8xR2-rescue:ESP32-DevKitC-MCU_Espressif
- U9: symbol Analog_ADC:ADS1299 -> ADS1299EMG8xR2-rescue:ADS1299-Analog_ADC
Changed lines of the file:
@@
 $EndDescr
 $Comp
-L MCU_Espressif:ESP32-DevKitC U13
+L ADS1299EMG8xR2-rescue:ESP32-DevKitC-MCU_Espressif U13
 U 1 1 5F7CFF1B
 P 8800 3800
@@
 P 3100 950
 F 0 "R19" V 3000 950 50  0000 C CNN
-F 1 "1M" V 3100 950 50  0000 C CNN
+F 1 "390k" V 3100 950 50  0000 C CNN
 F 2 "Resistor_SMD:R_0805_2012Metric_Pad1.20x1.40mm_HandSolder" V 3030 950 50  0001 C CNN
 F 3 "~" H 3100 950 50  0001 C CNN
@@
 U 1 1 5F88666F
 P 3100 1200
-F 0 "C14" V 3050 1100 50  0000 C CNN
-F 1 "1n5" V 3050 1300 50  0000 C CNN
+F 0 "C14" V 3050 1350 50  0000 C CNN
+F 1 "0.01uF" V 3150 1400 50  0000 C CNN
 F 2 "Capacitor_SMD:C_0805_2012Metric_Pad1.18x1.45mm_HandSolder" H 3138 1050 50  0001 C CNN
 F 3 "~" H 3100 1200 50  0001 C CNN
@@
 $EndSheet
 $Comp
-L Analog_ADC:ADS1299 U9
+L ADS1299EMG8xR2-rescue:ADS1299-Analog_ADC U9
 U 1 1 5F7CED44
 P 4800 3800
