File: hw_platform/ADS1299EMG8xR2/iamp.sch (KiCad schematic (older format))
At the start: 97 parts, among them U1 PJ-325-5P, U14 INA331, U15 INA331, U16 INA331, U17 INA331, U2 PJ-325-5P, U3 PJ-325-5P, U4 INA331, U5 INA331, U6 PJ-325-5P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

Commit message: Revision 4
Parts:
- added C1, C10, C2, C3, C6, C9: 0.1uF, Capacitor_SMD:C_0805_2012Metric_Pad1.18x1.45mm_HandSolder, symbol Device:C
Connections:
- net +5VA: now also C1.1, C10.1, C2.1, C3.1, C6.1, C9.1
- net GNDA: now also C1.2, C10.2, C2.2, C3.2, C6.2, C9.2
Other:
- moved on the sheet: R1, R6, R7, R8

Commit message: schematic verification
Parts:
- U1, U2, U3, U6, U7, U8: symbol Connector:PJ-325-5P -> ADS1299EMG8xR2-rescue:PJ-325-5P-Connector
- U14, U15, U16, U17, U4, U5: symbol Amplifier_Instrumentation:INA331 -> ADS1299EMG8xR2-rescue:INA331-Amplifier_Instrumentation
Changed lines of the file:
@@
 $EndComp
 $Comp
-L Connector:PJ-325-5P U?
+L ADS1299EMG8xR2-rescue:PJ-325-5P-Connector U?
 U 1 1 5FFE47AD
 P 1700 2700
@@
 $EndComp
 $Comp
-L Connector:PJ-325-5P U?
+L ADS1299EMG8xR2-rescue:PJ-325-5P-Connector U?
 U 1 1 60087200
 P 1700 1150
@@
 Connection ~ 3750 1200
 $Comp
-L Amplifier_Instrumentation:INA331 U?
+L ADS1299EMG8xR2-rescue:INA331-Amplifier_Instrumentation U?
 U 1 1 60087258
 P 3450 1200
@@
 $EndComp
 $Comp
-L Connector:PJ-325-5P U?
+L ADS1299EMG8xR2-rescue:PJ-325-5P-Connector U?
 U 1 1 600CBFB0
 P 1850 4250
@@
 $EndComp
 $Comp
-L Connector:PJ-325-5P U?
+L ADS1299EMG8xR2-rescue:PJ-325-5P-Connector U?
 U 1 1 5FFF3AFE
 P 1850 5850
@@
 $EndComp
 $Comp
-L Connector:PJ-325-5P U?
+L ADS1299EMG8xR2-rescue:PJ-325-5P-Connector U?
 U 1 1 606B6CA2
 P 6950 2650
@@
 Connection ~ 9200 2700
 $Comp
-L Amplifier_Instrumentation:INA331 U?
+L ADS1299EMG8xR2-rescue:INA331-Amplifier_Instrumentation U?
 U 1 1 606B6CFA
 P 8900 2700
@@
 $EndComp
 $Comp
-L Connector:PJ-325-5P U?
+L ADS1299EMG8xR2-rescue:PJ-325-5P-Connector U?
 U 1 1 608BE575
 P 7150 1150
@@
 Connection ~ 9200 1200
 $Comp
-L Amplifier_Instrumentation:INA331 U?
+L ADS1299EMG8xR2-rescue:INA331-Amplifier_Instrumentation U?
 U 1 1 608BE5CD
 P 8900 1200
@@
 Connection ~ 3750 2750
 $Comp
-L Amplifier_Instrumentation:INA331 U?
+L ADS1299EMG8xR2-rescue:INA331-Amplifier_Instrumentation U?
 U 1 1 5FFE47F1
 P 3450 2750
@@
 $EndComp
 $Comp
-L Amplifier_Instrumentation:INA331 U?
+L ADS1299EMG8xR2-rescue:INA331-Amplifier_Instrumentation U?
 U 1 1 6062C446
 P 3950 4450
@@
 	2250 6350 2450 6350
 $Comp
-L Amplifier_Instrumentation:INA331 U?
+L ADS1299EMG8xR2-rescue:INA331-Amplifier_Instrumentation U?
 U 1 1 608CF427
 P 3950 6050
