File: hw_platform/MYOCELL2/power_supply.kicad_sch (KiCad schematic)
At the start: 21 parts, among them J2 Battery Connector JC2, J3 Battery Connector JC2, Q2 DMG3404L, SW1 SW_Nidec_CAS-120A1, U10 AP2112K-3.3, U17 MCP73831-2-OT, U9 AP2112K-3.3

Commit message: working on schematic:
Parts:
- removed J2, J3: Battery Connector JC2, Connector_JST:JST_EH_B2B-EH-A_1x02_P2.50mm_Vertical, symbol Connector_Generic:Conn_01x02
- renumbered C35 to C17, C39 to C18, C34 to C19, C38 to C20, U10 to U6, U9 to U7
Connections:
- net BAT: now reaches C51.1, Q2.2 (S), R44.2, U17.3 (V_{BAT})
Other:
- note removed: "To battery"
- note removed: "To next board in chain"
- moved on the sheet: C50, C51, C52, D2, D3, Q2, R41, R42, R43, R44, R45, SW1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
