File: hw_platform/simulate/Analogue_interfaces/simulate.kicad_sch (KiCad schematic)
At the start: 23 parts, among them U1 INA331, U2 OPA340NA

Commit message: GND replaced with simulation GND
Parts:
- removed V1: AC 0.1, symbol pspice:VSOURCE
- removed V3: 3.3, symbol pspice:VSOURCE
- removed V4: 2.4, symbol pspice:VSOURCE
- added V2: 2.4, symbol Simulation_SPICE:VDC
- added V3: 3.3, symbol Simulation_SPICE:VDC
- added V4: VSIN, symbol Simulation_SPICE:VSIN
Connections:
- net GND: no longer R14.2, R8.2, U1.4 (V-), U2.2 (V-)
- net GREEN: now also V4.1
- net RED: now also V4.2
- net Vs: now also V3.1
- net at R7.1: now also V2.1
- new net 0: R14.2, R8.2, U1.4 (V-), U2.2 (V-), V2.2, V3.2
